File: IRIS-7/Precharge/pre-charge.kicad_pcb (KiCad board)
At the start: 2 copper layers, 56 x 36 mm, 36 parts, among them IC1 LM324, IC3 LMR16006, P1 CONN_01X03, P2 CONN_01X02, Q1 DMP3099L

Commit message: Minor tweaks before OK2FAB
Parts:
- added G***: LOGO, IRIS_Logos:IRIS_Logo_13.5, B.Cu at (146.0, 123.5)
Other:
- board text added: "JP2 (UVLO)"
- board text added: "Relay"
- board text added: "Rev A"
- board text added: "TH"
- board text added: "UVLO EN: Short"
- board text added: "V"
- board text removed: "Byron's Comments: - Add IRIS logo (I can help you with this)"
- board text removed: "Vrelay"

Commit message: Make final changes before fab release
Parts:
- added C5: 100nF, Capacitors_SMD:C_0805, B.Cu at (172.5, 104.5)
- added C6: 1nF, Capacitors_SMD:C_0805, B.Cu at (166.5, 104.5)
- added C7: 100nF, Capacitors_SMD:C_0805, B.Cu at (164.5, 104.5)
- added D3: Blue, LEDs:LED_0805, F.Cu at (175.5, 130.0)
- added D4: Orange, LEDs:LED_0805, F.Cu at (177.5, 130.0)
- added IC2: MAX6001, TO_SOT_Packages_SMD:SOT-23, B.Cu at (169.5, 104.5)
- added R18: 1k, Resistors_SMD:R_0805, B.Cu at (174.5, 104.5)
- added R19: 1k, Resistors_SMD:R_0805, F.Cu at (153.5, 118.8)
- moved JP1 5.08 mm to (150.6, 102.3), turned to 0 degrees
Connections:
- R10 pad 2: Net-(JP1-Pad3) -> Net-(JP1-Pad1)
- R11 pad 1: Net-(JP1-Pad1) -> Net-(JP1-Pad3)
- R12 pad 2: Net-(JP1-Pad1) -> Net-(JP1-Pad3)
- R9 pad 1: Net-(JP1-Pad3) -> Net-(JP1-Pad1)
Routing:
- net Net-(D4-Pad2): track 0.00 -> 30.1 mm, vias 0 -> 2
- net Net-(D3-Pad2): track 0.00 -> 23.9 mm, vias 0 -> 1
- net Net-(JP1-Pad1): track 9.12 -> 23.9 mm
- net Net-(JP1-Pad3): track 23.8 -> 9.12 mm
- net +12V: track 14.7 -> 28.4 mm
- net /Vref: track 0.00 -> 8.73 mm, vias 0 -> 1
- net /Relay_Gate: track 8.68 -> 14.3 mm
- net /Vbat: track 55.4 -> 52.1 mm
Other:
- net class 1A: clearance 0.15 -> 0.2
- net class Default: clearance 0.15 -> 0.2
- rule trace_clearance: 0.15 -> 0.2
- board text added: "Please place any manufacturing marks in this area"
